Commit message: wheel-track#2

File: esaul_description/urdf/esaul.xacro (robot description, xacro)
@@ -6,9 +6,9 @@
   <xacro:property name="chassis_height" value="0.13" />
   <xacro:property name="track_mass" value="0.3" />
-  <xacro:property name="track_rad" value="0.04" />
+  <xacro:property name="track_rad" value="0.03" />
   <xacro:property name="track_length" value="0.04" />
   <xacro:property name="box_length" value="0.4" />
-  <xacro:property name="box_width" value="0.04" />
-  <xacro:property name="box_height" value="0.08" />
+  <xacro:property name="box_width" value="0.03" />
+  <xacro:property name="box_height" value="0.06" />
    <xacro:property name="wheel_mass" value="1" />
   <xacro:property name="wheel_friction" value="1.75" />
@@ -49,7 +49,7 @@
       <xacro:insert_block name="origin"/>
       <mass value="${mass}"/>
-      <inertia ixx="${0.01 + (mass * h * h)/12 + (mass * r * r)/4}" ixy="0.0" ixz="0.0"
-               iyy="${0.01 + (mass * h * h)/12 + (mass * r * r)/4}" iyz="0.0"
-               izz="${0.01 + mass / 2 * r * r}" />
+      <inertia ixx="${(mass * h * h)/12 + (mass * r * r)/4}" ixy="0.0" ixz="0.0"
+               iyy="${(mass * h * h)/12 + (mass * r * r)/4}" iyz="0.0"
+               izz="${mass / 2 * r * r}" />
     </inertial>
   </xacro:macro>
@@ -95,6 +95,6 @@
     </link>
     <gazebo reference="${name}">
-      <mu1>1</mu1>
-      <mu2>1</mu2>
+      <mu1>0</mu1>
+      <mu2>0</mu2>
       <material>Gazebo/Black</material>
     </gazebo>

Commit message: wheel-track#3

File: esaul_description/urdf/esaul.xacro (robot description, xacro)
@@ -57,4 +57,5 @@
   <link name="link_chassis">
     <collision name="collision_chassis">
+      <!-- <origin rpy="0 0 0" xyz="0 0 ${track_rad}"/> -->
       <geometry>
         <box size="${chassis_length} ${chassis_width} ${chassis_height}"/>
@@ -62,9 +63,8 @@
     </collision>
     <visual>
-      <origin rpy="0 0 0" xyz="0 0 ${track_rad}"/>
+      <!-- <origin rpy="0 0 0" xyz="0 0 ${track_rad}"/> -->
       <geometry>
         <box size="${chassis_length} ${chassis_width} ${chassis_height}"/>
       </geometry>
-      <material name="blue"/>
     </visual>
     <xacro:solid_cuboid_inertial
@@ -77,4 +77,5 @@
     <link name="${name}">
       <collision name="collision_left_track">
+        <origin rpy="0 0 0" xyz="0 0 0"/>
         <geometry>
           <box size="${box_length} ${box_width} ${box_height}"/>
@@ -124,6 +125,6 @@
       <mu2>1.5</mu2>
       <material>Gazebo/Black</material>
-      <!-- <kp>10000000</kp> -->
-      <!-- <kd>1</kd> -->
+      <kp>10000000</kp>
+      <kd>1</kd>
     </gazebo>
   </xacro:macro>
@@ -160,5 +161,5 @@
   </xacro:macro>
   <xacro:link_track name="link_right" />
-	<xacro:joint_track name="joint_right" child="link_right" origin_xyz="0 ${-chassis_width/2-box_width/2} ${-track_rad}" />
+	<xacro:joint_track name="joint_right" child="link_right" origin_xyz="0 ${-chassis_width/2-box_width/2} ${-2*box_width}" />
   <xacro:link_wheel name="right_wheel_1" />
 	<xacro:joint_wheel_right name="joint_right_wheel_1" child="right_wheel_1" origin_xyz="${box_length/2} 0 0" />
@@ -170,5 +171,5 @@
 	<xacro:joint_wheel_right name="joint_right_wheel_4" child="right_wheel_4" origin_xyz="${-box_length/2} 0 0" />
   <xacro:link_track name="link_left" />
-	<xacro:joint_track name="joint_left" child="link_left" origin_xyz="0 ${chassis_width/2+box_width/2} ${-track_rad}" />
+	<xacro:joint_track name="joint_left" child="link_left" origin_xyz="0 ${chassis_width/2+box_width/2} ${-2*box_width}" />
   <xacro:link_wheel name="left_wheel_1" />
 	<xacro:joint_wheel_left name="joint_left_wheel_1" child="left_wheel_1" origin_xyz="${box_length/2} 0 0" />

Commit message: wheel-track#4

File: esaul_description/urdf/esaul.xacro (robot description, xacro)
@@ -8,8 +8,8 @@
   <xacro:property name="track_rad" value="0.03" />
   <xacro:property name="track_length" value="0.04" />
-  <xacro:property name="box_length" value="0.4" />
+  <xacro:property name="box_length" value="0.35" />
   <xacro:property name="box_width" value="0.03" />
   <xacro:property name="box_height" value="0.06" />
-   <xacro:property name="wheel_mass" value="1" />
+   <xacro:property name="wheel_mass" value="10" />
   <xacro:property name="wheel_friction" value="1.75" />
   <!-- INERTIAL MACROS -->
@@ -27,9 +27,9 @@
       <xacro:insert_block name="origin"/>
       <mass value="${mass}"/>
-      <inertia ixx="${mass * (width * width + height * height) / 12}"
+      <inertia ixx="${0.01+ mass * (width * width + height * height) / 12}"
                ixy="0" ixz="0"
-               iyy="${mass * (length * length + height * height) / 12}"
+               iyy="${0.01+ mass * (length * length + height * height) / 12}"
                iyz="0"
-               izz="${mass * (width * width + length * length) / 12}"/>
+               izz="${0.01+ mass * (width * width + length * length) / 12}"/>
     </inertial>
   </xacro:macro>
@@ -161,23 +161,19 @@
   </xacro:macro>
   <xacro:link_track name="link_right" />
-	<xacro:joint_track name="joint_right" child="link_right" origin_xyz="0 ${-chassis_width/2-box_width/2} ${-2*box_width}" />
+	<xacro:joint_track name="joint_right" child="link_right" origin_xyz="0 ${-chassis_width/2-box_width/1.5} ${-2*box_width}" />
   <xacro:link_wheel name="right_wheel_1" />
 	<xacro:joint_wheel_right name="joint_right_wheel_1" child="right_wheel_1" origin_xyz="${box_length/2} 0 0" />
   <xacro:link_wheel name="right_wheel_2" />
-	<xacro:joint_wheel_right name="joint_right_wheel_2" child="right_wheel_2" origin_xyz="${box_length/6} 0 0" />
+	<xacro:joint_wheel_right name="joint_right_wheel_2" child="right_wheel_2" origin_xyz="0 0 0" />
   <xacro:link_wheel name="right_wheel_3" />
-	<xacro:joint_wheel_right name="joint_right_wheel_3" child="right_wheel_3" origin_xyz="${-box_length/6} 0 0" />
-  <xacro:link_wheel name="right_wheel_4" />
-	<xacro:joint_wheel_right name="joint_right_wheel_4" child="right_wheel_4" origin_xyz="${-box_length/2} 0 0" />
+	<xacro:joint_wheel_right name="joint_right_wheel_3" child="right_wheel_3" origin_xyz="${-box_length/2} 0 0" />
   <xacro:link_track name="link_left" />
-	<xacro:joint_track name="joint_left" child="link_left" origin_xyz="0 ${chassis_width/2+box_width/2} ${-2*box_width}" />
+	<xacro:joint_track name="joint_left" child="link_left" origin_xyz="0 ${chassis_width/2+box_width/1.5} ${-2*box_width}" />
   <xacro:link_wheel name="left_wheel_1" />
 	<xacro:joint_wheel_left name="joint_left_wheel_1" child="left_wheel_1" origin_xyz="${box_length/2} 0 0" />
   <xacro:link_wheel name="left_wheel_2" />
-	<xacro:joint_wheel_left name="joint_left_wheel_2" child="left_wheel_2" origin_xyz="${box_length/6} 0 0" />
+	<xacro:joint_wheel_left name="joint_left_wheel_2" child="left_wheel_2" origin_xyz="0 0 0" />
   <xacro:link_wheel name="left_wheel_3" />
-	<xacro:joint_wheel_left name="joint_left_wheel_3" child="left_wheel_3" origin_xyz="${-box_length/6} 0 0" />
-  <xacro:link_wheel name="left_wheel_4" />
-	<xacro:joint_wheel_left name="joint_left_wheel_4" child="left_wheel_4" origin_xyz="${-box_length/2} 0 0" />
+	<xacro:joint_wheel_left name="joint_left_wheel_3" child="left_wheel_3" origin_xyz="${-box_length/2} 0 0" />
   	<gazebo>
     		<plugin name="ModelPlugin" filename="libesaul_description.so" >
@@ -189,9 +185,6 @@
             <joint_left3>joint_left_wheel_3</joint_left3>
             <joint_right3>joint_right_wheel_3</joint_right3>
-            <joint_left4>joint_left_wheel_4</joint_left4>
-            <joint_right4>joint_right_wheel_4</joint_right4>
             <width_chassis>${chassis_width}</width_chassis>
-            <link_r>link_right</link_r>
-            <link_l>link_left</link_l>
+            <wh_rad>${track_rad}</wh_rad>
    		 </plugin>
 	</gazebo>

Commit message: lidar with teleop

File: esaul_description/urdf/esaul.xacro (robot description, xacro)
@@ -11,5 +11,8 @@
   <xacro:property name="box_width" value="0.03" />
   <xacro:property name="box_height" value="0.06" />
-   <xacro:property name="wheel_mass" value="10" />
+  <xacro:property name="wheel_mass" value="10" />
+  <xacro:property name="lidar_mass" value="0.1" />
+  <xacro:property name="lidar_height" value="0.02"/>
+  <xacro:property name="lidar_radius" value="0.04"/>
   <xacro:property name="wheel_friction" value="1.75" />
   <!-- INERTIAL MACROS -->
@@ -160,4 +163,95 @@
     </joint>
   </xacro:macro>
+<!--
+  <link name="laser_frame">
+    <xacro:solid_cylinder_inertial
+        r="${lidar_radius}" h="${lidar_height}"
+        mass="${lidar_mass}" >
+      <origin xyz="0 0 0" rpy="0 0 0" />
+    </xacro:solid_cylinder_inertial>
+    <collision>
+      <origin xyz="0 0 0" rpy="0 0 0" />
+      <geometry>
+        <cylinder length="${lidar_height}" radius="${lidar_radius}"/>
+      </geometry>
+    </collision>
+    <visual>
+      <origin xyz="0 0 0" rpy="0 0 0" />
+      <geometry>
+        <cylinder length="${lidar_height}" radius="${lidar_radius}"/>
+      </geometry>
+    </visual>
+  </link>
+  <gazebo reference="laser_frame">
+    <material>Gazebo/Red</material>
+  </gazebo>
+  <joint name="laser_joint" type="fixed">
+    <child link="laser_frame" />
+    <parent link="link_chassis" />
+    <origin xyz="0 0 ${chassis_height/2 + lidar_height/2}" />
+  </joint>
+ -->
+  <!-- Hokuyo Laser -->
+  <link name="lidar_link">
+    <xacro:solid_cylinder_inertial
+        r="${lidar_radius}" h="${lidar_height}"
+        mass="${lidar_mass}" >
+      <origin xyz="0 0 0" rpy="0 0 0" />
+    </xacro:solid_cylinder_inertial>
+    <collision>
+      <origin xyz="0 0 0" rpy="0 0 0"/>
+      <geometry>
+        <cylinder length="${lidar_height}" radius="${lidar_radius}"/>
+      </geometry>
+    </collision>
+    <visual>
+      <origin xyz="0 0 0" rpy="0 0 0"/>
+      <geometry>
+        <cylinder length="${lidar_height}" radius="${lidar_radius}"/>
+      </geometry>
+    </visual>
+  </link>
+  <gazebo reference="lidar_link">
+    <material>Gazebo/Red</material>
+    <sensor type="ray" name="head_hokuyo_sensor">
+      <pose>0 0 0 0 0 0</pose>
+      <visualize>true</visualize>
+      <update_rate>40</update_rate>
+      <ray>
+        <scan>
+          <horizontal>
+            <samples>720</samples>
+            <resolution>1</resolution>
+            <min_angle>-3.14</min_angle>
+            <max_angle>3.14</max_angle>
+          </horizontal>
+        </scan>
+        <range>
+          <min>0.10</min>
+          <max>30.0</max>
+          <resolution>0.01</resolution>
+        </range>
+        <noise>
+          <type>gaussian</type>
+          <!-- Noise parameters based on published spec for Hokuyo laser
+               achieving "+-30mm" accuracy at range < 10m.  A mean of 0.0m and
+               stddev of 0.01m will put 99.7% of samples within 0.03m of the true
+               reading. -->
+          <mean>0.0</mean>
+          <stddev>0.01</stddev>
+        </noise>
+      </ray>
+      <plugin name="gazebo_ros_head_hokuyo_controller" filename="libgazebo_ros_laser.so">
+        <topicName>/eSAUl/laser/scan</topicName>
+        <frameName>lidar_link</frameName>
+      </plugin>
+    </sensor>
+  </gazebo>
+  <joint name="lidar_joint" type="fixed">
+    <axis xyz="0 1 0" />
+    <origin xyz="0 0 ${chassis_height/2 + lidar_height/2}" rpy="0 0 0"/>
+    <parent link="link_chassis"/>
+    <child link="lidar_link"/>
+  </joint>
   <xacro:link_track name="link_right" />
 	<xacro:joint_track name="joint_right" child="link_right" origin_xyz="0 ${-chassis_width/2-box_width/1.5} ${-2*box_width}" />

Commit message: gmapping and tf

File: esaul_description/urdf/esaul.xacro (robot description, xacro)
@@ -30,9 +30,9 @@
       <xacro:insert_block name="origin"/>
       <mass value="${mass}"/>
-      <inertia ixx="${0.01+ mass * (width * width + height * height) / 12}"
+      <inertia ixx="${mass * (width * width + height * height) / 12}"
                ixy="0" ixz="0"
-               iyy="${0.01+ mass * (length * length + height * height) / 12}"
+               iyy="${mass * (length * length + height * height) / 12}"
                iyz="0"
-               izz="${0.01+ mass * (width * width + length * length) / 12}"/>
+               izz="${mass * (width * width + length * length) / 12}"/>
     </inertial>
   </xacro:macro>
@@ -58,5 +58,5 @@
   </xacro:macro>
   <!-- INERTIAL MACROS END -->
-  <link name="link_chassis">
+  <link name="base_link">
     <collision name="collision_chassis">
       <!-- <origin rpy="0 0 0" xyz="0 0 ${track_rad}"/> -->
@@ -158,5 +158,5 @@
       <origin rpy="0 0 0" xyz="${origin_xyz}"/>
       <child link="${child}"/>
-      <parent link="link_chassis"/>
+      <parent link="base_link"/>
       <axis rpy="0 0 0" xyz="0 1 0"/>
       <joint_properties damping="1.0" friction="0.0"/>
@@ -188,5 +188,5 @@
   <joint name="laser_joint" type="fixed">
     <child link="laser_frame" />
-    <parent link="link_chassis" />
+    <parent link="base_link" />
     <origin xyz="0 0 ${chassis_height/2 + lidar_height/2}" />
   </joint>
@@ -216,5 +216,5 @@
     <sensor type="ray" name="head_hokuyo_sensor">
       <pose>0 0 0 0 0 0</pose>
-      <visualize>true</visualize>
+      <visualize>false</visualize>
       <update_rate>40</update_rate>
       <ray>
@@ -251,5 +251,5 @@
     <axis xyz="0 1 0" />
     <origin xyz="0 0 ${chassis_height/2 + lidar_height/2}" rpy="0 0 0"/>
-    <parent link="link_chassis"/>
+    <parent link="base_link"/>
     <child link="lidar_link"/>
   </joint>

Commit message: encoder

File: esaul_description/urdf/esaul.xacro (robot description, xacro)
@@ -1,5 +1,5 @@
 <?xml version="1.0" ?>
 <robot name="eSAUl" xmlns:xacro="http://www.ros.org/wiki/xacro">
-  <xacro:property name="chassis_mass" value="20" />
+  <xacro:property name="chassis_mass" value="40" />
   <xacro:property name="chassis_length" value="0.45" />
   <xacro:property name="chassis_width" value="0.22" />

Commit message: gmapping

File: esaul_description/urdf/esaul.xacro (robot description, xacro)
@@ -1,4 +1,5 @@
 <?xml version="1.0" ?>
 <robot name="eSAUl" xmlns:xacro="http://www.ros.org/wiki/xacro">
+  <xacro:property name="M_PI" value="3.1415926535897931" />
   <xacro:property name="chassis_mass" value="40" />
   <xacro:property name="chassis_length" value="0.45" />
@@ -6,9 +7,9 @@
   <xacro:property name="chassis_height" value="0.13" />
   <xacro:property name="track_mass" value="0.3" />
-  <xacro:property name="track_rad" value="0.03" />
-  <xacro:property name="track_length" value="0.04" />
-  <xacro:property name="box_length" value="0.35" />
+  <xacro:property name="track_rad" value="0.04" />
+  <xacro:property name="track_length" value="0.03" />
+  <xacro:property name="box_length" value="0.4" />
   <xacro:property name="box_width" value="0.03" />
-  <xacro:property name="box_height" value="0.06" />
+  <xacro:property name="box_height" value="0.08" />
   <xacro:property name="wheel_mass" value="10" />
   <xacro:property name="lidar_mass" value="0.1" />
@@ -24,4 +25,12 @@
                izz="0.01"/>
       </inertial>
+  </xacro:macro>
+  <xacro:macro name="default_inertial" params="mass">
+    <inertial>
+      <mass value="${mass}" />
+    <inertia ixx="1.0" ixy="0.0" ixz="0.0"
+             iyy="1.0" iyz="0.0"
+             izz="1.0" />
+    </inertial>
   </xacro:macro>
   <xacro:macro name="solid_cuboid_inertial"
@@ -37,14 +46,4 @@
     </inertial>
   </xacro:macro>
-  <!-- <xacro:macro name="solid_cylinder_inertial"
-               params="r h mass *origin">
-    <inertial>
-      <xacro:insert_block name="origin"/>
-      <mass value="${mass}"/>
-      <inertia ixx="${mass / 12 * (3 * r * r + h * h)}" ixy="0.0" ixz="0.0"
-               iyy="${mass / 12 * (3 * r * r + h * h)}" iyz="0.0"
-               izz="${mass / 2 * r * r}" />
-    </inertial>
-  </xacro:macro> -->
     <xacro:macro name="solid_cylinder_inertial"
                params="r h mass *origin">
@@ -80,5 +79,5 @@
     <link name="${name}">
       <collision name="collision_left_track">
-        <origin rpy="0 0 0" xyz="0 0 0"/>
+        <origin rpy="0 0 0" xyz="0 0 0.01"/>
         <geometry>
           <box size="${box_length} ${box_width} ${box_height}"/>
@@ -86,5 +85,5 @@
       </collision>
       <visual>
-        <origin rpy="0 0 0" xyz="0 0 0"/>
+        <origin rpy="0 0 0" xyz="0 0 0.01"/>
         <geometry>
           <box size="${box_length} ${box_width} ${box_height}"/>
@@ -125,6 +124,6 @@
     </link>
     <gazebo reference="${name}">
-      <mu1>1.5</mu1>
-      <mu2>1.5</mu2>
+      <mu1>3</mu1>
+      <mu2>3</mu2>
       <material>Gazebo/Black</material>
       <kp>10000000</kp>
@@ -139,6 +138,4 @@
       <axis rpy="0 0 0" xyz="0 1 0"/>
       <limit effort="10000" velocity="1000"/>
-      <!-- <use_parent_model_frame>1</use_parent_model_frame> -->
-      <!-- <joint_properties damping="1.0" friction="1.0"/> -->
     </joint>
   </xacro:macro>
@@ -150,6 +147,4 @@
       <axis rpy="0 0 0" xyz="0 1 0"/>
       <limit effort="10000" velocity="1000"/>
-      <!-- <use_parent_model_frame>1</use_parent_model_frame> -->
-      <!-- <joint_properties damping="1.0" friction="1.0"/> -->
     </joint>
   </xacro:macro>
@@ -163,34 +158,4 @@
     </joint>
   </xacro:macro>
-<!--
-  <link name="laser_frame">
-    <xacro:solid_cylinder_inertial
-        r="${lidar_radius}" h="${lidar_height}"
-        mass="${lidar_mass}" >
-      <origin xyz="0 0 0" rpy="0 0 0" />
-    </xacro:solid_cylinder_inertial>
-    <collision>
-      <origin xyz="0 0 0" rpy="0 0 0" />
-      <geometry>
-        <cylinder length="${lidar_height}" radius="${lidar_radius}"/>
-      </geometry>
-    </collision>
-    <visual>
-      <origin xyz="0 0 0" rpy="0 0 0" />
-      <geometry>
-        <cylinder length="${lidar_height}" radius="${lidar_radius}"/>
-      </geometry>
-    </visual>
-  </link>
-  <gazebo reference="laser_frame">
-    <material>Gazebo/Red</material>
-  </gazebo>
-  <joint name="laser_joint" type="fixed">
-    <child link="laser_frame" />
-    <parent link="base_link" />
-    <origin xyz="0 0 ${chassis_height/2 + lidar_height/2}" />
-  </joint>
- -->
-  <!-- Hokuyo Laser -->
   <link name="lidar_link">
     <xacro:solid_cylinder_inertial
@@ -234,8 +199,4 @@
         <noise>
           <type>gaussian</type>
-          <!-- Noise parameters based on published spec for Hokuyo laser
-               achieving "+-30mm" accuracy at range < 10m.  A mean of 0.0m and
-               stddev of 0.01m will put 99.7% of samples within 0.03m of the true
-               reading. -->
           <mean>0.0</mean>
           <stddev>0.01</stddev>
@@ -244,5 +205,5 @@
       <plugin name="gazebo_ros_head_hokuyo_controller" filename="libgazebo_ros_laser.so">
         <topicName>/eSAUl/laser/scan</topicName>
-        <frameName>lidar_link</frameName>
+        <frameName>laser_frame</frameName>
       </plugin>
     </sensor>
@@ -254,29 +215,55 @@
     <child link="lidar_link"/>
   </joint>
+ <xacro:macro name="support_wheel" params="parent location *origin">
+    <link name="support_wheel_${location}_link">
+      <visual>
+        <origin xyz="0 0 0" rpy="0 0 0" />
+        <geometry>
+          <mesh filename="package://caster_description/mesh/support_wheel.stl" />
+        </geometry>
+        <material name="">
+          <color rgba="0.3 0.3 0.3 1.0" />>
+        </material>
+      </visual>
+      <collision>
+        <origin xyz="0 0 0" rpy="0 0 0" />
+        <geometry>
+          <mesh filename="package://caster_description/mesh/support_wheel.stl" />
+        </geometry>
+      </collision>
+      <xacro:default_inertial mass="5" />
+    </link>
+    <joint name="support_wheel_${location}_joint" type="fixed">
+      <xacro:insert_block name="origin" />
+      <parent link="${parent}" />
+      <child link="support_wheel_${location}_link" />
+      <!-- <axis xyz="0 0 1" /> -->
+    </joint>
+  </xacro:macro>
   <xacro:link_track name="link_right" />
 	<xacro:joint_track name="joint_right" child="link_right" origin_xyz="0 ${-chassis_width/2-box_width/1.5} ${-2*box_width}" />
-  <xacro:link_wheel name="right_wheel_1" />
-	<xacro:joint_wheel_right name="joint_right_wheel_1" child="right_wheel_1" origin_xyz="${box_length/2} 0 0" />
-  <xacro:link_wheel name="right_wheel_2" />
-	<xacro:joint_wheel_right name="joint_right_wheel_2" child="right_wheel_2" origin_xyz="0 0 0" />
-  <xacro:link_wheel name="right_wheel_3" />
-	<xacro:joint_wheel_right name="joint_right_wheel_3" child="right_wheel_3" origin_xyz="${-box_length/2} 0 0" />
+  <xacro:link_wheel name="right_wheel" />
+	<xacro:joint_wheel_right name="joint_right_wheel" child="right_wheel" origin_xyz="0 0 0" />
   <xacro:link_track name="link_left" />
 	<xacro:joint_track name="joint_left" child="link_left" origin_xyz="0 ${chassis_width/2+box_width/1.5} ${-2*box_width}" />
-  <xacro:link_wheel name="left_wheel_1" />
-	<xacro:joint_wheel_left name="joint_left_wheel_1" child="left_wheel_1" origin_xyz="${box_length/2} 0 0" />
-  <xacro:link_wheel name="left_wheel_2" />
-	<xacro:joint_wheel_left name="joint_left_wheel_2" child="left_wheel_2" origin_xyz="0 0 0" />
-  <xacro:link_wheel name="left_wheel_3" />
-	<xacro:joint_wheel_left name="joint_left_wheel_3" child="left_wheel_3" origin_xyz="${-box_length/2} 0 0" />
-  	<gazebo>
+  <xacro:link_wheel name="left_wheel" />
+	<xacro:joint_wheel_left name="joint_left_wheel" child="left_wheel" origin_xyz="0 0 0" />
+  <xacro:support_wheel parent="link_left" location="left_1">
+    <origin xyz="${box_length/2} 0 0.028" rpy="0 0 0" />
+  </xacro:support_wheel>
+  <xacro:support_wheel parent="link_left" location="left_2">
+    <origin xyz="${-box_length/2} 0 0.028" rpy="0 0 0" />
+  </xacro:support_wheel>
+  <xacro:support_wheel parent="link_right" location="right_1">
+    <origin xyz="${box_length/2} 0 0.028" rpy="0 0 0" />
+  </xacro:support_wheel>
+  <xacro:support_wheel parent="link_right" location="right_2">
+    <origin xyz="${-box_length/2} 0 0.028" rpy="0 0 0" />
+  </xacro:support_wheel>
+  <gazebo>
     		<plugin name="ModelPlugin" filename="libesaul_description.so" >
-      			<robotName>eSAUl</robotName>
-            <joint_left1>joint_left_wheel_1</joint_left1>
-            <joint_right1>joint_right_wheel_1</joint_right1>
-            <joint_left2>joint_left_wheel_2</joint_left2>
-            <joint_right2>joint_right_wheel_2</joint_right2>
-            <joint_left3>joint_left_wheel_3</joint_left3>
-            <joint_right3>joint_right_wheel_3</joint_right3>
+      		<robotName>eSAUl</robotName>
+            <joint_left>joint_left_wheel</joint_left>
+            <joint_right>joint_right_wheel</joint_right>
             <width_chassis>${chassis_width}</width_chassis>
             <wh_rad>${track_rad}</wh_rad>
