Commit message: fix and folder esaul_software

File: esaul_description/urdf/esaul.xacro (robot description, xacro)
@@ -1,4 +1,7 @@
 <?xml version="1.0" ?>
 <robot name="eSAUl" xmlns:xacro="http://www.ros.org/wiki/xacro">
+  <xacro:include filename="$(find esaul_description)/urdf/track.xacro" />
+  <xacro:include filename="$(find esaul_description)/urdf/wheel.xacro" />
+  <xacro:include filename="$(find esaul_software)/urdf/lidar.xacro" />
   <xacro:property name="M_PI" value="3.1415926535897931" />
   <xacro:property name="chassis_mass" value="40" />
@@ -6,14 +9,4 @@
   <xacro:property name="chassis_width" value="0.22" />
   <xacro:property name="chassis_height" value="0.13" />
-  <xacro:property name="track_mass" value="0.3" />
-  <xacro:property name="track_rad" value="0.04" />
-  <xacro:property name="track_length" value="0.03" />
-  <xacro:property name="box_length" value="0.4" />
-  <xacro:property name="box_width" value="0.03" />
-  <xacro:property name="box_height" value="0.08" />
-  <xacro:property name="wheel_mass" value="10" />
-  <xacro:property name="lidar_mass" value="0.1" />
-  <xacro:property name="lidar_height" value="0.02"/>
-  <xacro:property name="lidar_radius" value="0.04"/>
   <xacro:property name="wheel_friction" value="1.75" />
   <!-- INERTIAL MACROS -->
@@ -46,14 +39,4 @@
     </inertial>
   </xacro:macro>
-    <xacro:macro name="solid_cylinder_inertial"
-               params="r h mass *origin">
-    <inertial>
-      <xacro:insert_block name="origin"/>
-      <mass value="${mass}"/>
-      <inertia ixx="${(mass * h * h)/12 + (mass * r * r)/4}" ixy="0.0" ixz="0.0"
-               iyy="${(mass * h * h)/12 + (mass * r * r)/4}" iyz="0.0"
-               izz="${mass / 2 * r * r}" />
-    </inertial>
-  </xacro:macro>
   <!-- INERTIAL MACROS END -->
   <link name="base_link">
@@ -76,169 +59,4 @@
     </xacro:solid_cuboid_inertial>
   </link>
-  <xacro:macro name="link_track" params="name">
-    <link name="${name}">
-      <collision name="collision_left_track">
-        <origin rpy="0 0 0" xyz="0 0 0.01"/>
-        <geometry>
-          <box size="${box_length} ${box_width} ${box_height}"/>
-        </geometry>
-      </collision>
-      <visual>
-        <origin rpy="0 0 0" xyz="0 0 0.01"/>
-        <geometry>
-          <box size="${box_length} ${box_width} ${box_height}"/>
-        </geometry>
-        <material name="black"/>
-      </visual>
-      <xacro:solid_cuboid_inertial
-            length="${box_length}" width="${box_width}"
-            height="${box_height}" mass="${track_mass}">
-        <origin xyz="0 0 0" rpy="0 0 0" />
-      </xacro:solid_cuboid_inertial>
-    </link>
-    <gazebo reference="${name}">
-      <mu1>0</mu1>
-      <mu2>0</mu2>
-      <material>Gazebo/Black</material>
-    </gazebo>
-  </xacro:macro>
-  <xacro:macro name="link_wheel" params="name">
-    <link name="${name}">
-      <xacro:solid_cylinder_inertial
-          r="${track_rad}" h="${track_length}"
-          mass="${wheel_mass}" >
-        <origin xyz="0 0 0" rpy="0 0 0" />
-      </xacro:solid_cylinder_inertial>
-      <collision name="link_right_wheel_collision">
-        <origin rpy="0 1.5707 1.5707" xyz="0 0 0"/>
-        <geometry>
-          <cylinder length="${track_length}" radius="${track_rad}"/>
-        </geometry>
-      </collision>
-      <visual name="${name}_visual">
-        <origin rpy="0 1.5707 1.5707" xyz="0 0 0"/>
-        <geometry>
-          <cylinder length="${track_length}" radius="${track_rad}"/>
-        </geometry>
-      </visual>
-    </link>
-    <gazebo reference="${name}">
-      <mu1>3</mu1>
-      <mu2>3</mu2>
-      <material>Gazebo/Black</material>
-      <kp>10000000</kp>
-      <kd>1</kd>
-    </gazebo>
-  </xacro:macro>
-  <xacro:macro name="joint_wheel_right" params="name child origin_xyz">
-    <joint name="${name}" type="continuous">
-      <origin rpy="0 0 0" xyz="${origin_xyz}"/>
-      <child link="${child}"/>
-      <parent link="link_right"/>
-      <axis rpy="0 0 0" xyz="0 1 0"/>
-      <limit effort="10000" velocity="1000"/>
-    </joint>
-  </xacro:macro>
-    <xacro:macro name="joint_wheel_left" params="name child origin_xyz">
-    <joint name="${name}" type="continuous">
-      <origin rpy="0 0 0" xyz="${origin_xyz}"/>
-      <child link="${child}"/>
-      <parent link="link_left"/>
-      <axis rpy="0 0 0" xyz="0 1 0"/>
-      <limit effort="10000" velocity="1000"/>
-    </joint>
-  </xacro:macro>
-  <xacro:macro name="joint_track" params="name child origin_xyz">
-    <joint name="${name}" type="fixed">
-      <origin rpy="0 0 0" xyz="${origin_xyz}"/>
-      <child link="${child}"/>
-      <parent link="base_link"/>
-      <axis rpy="0 0 0" xyz="0 1 0"/>
-      <joint_properties damping="1.0" friction="0.0"/>
-    </joint>
-  </xacro:macro>
-  <link name="lidar_link">
-    <xacro:solid_cylinder_inertial
-        r="${lidar_radius}" h="${lidar_height}"
-        mass="${lidar_mass}" >
-      <origin xyz="0 0 0" rpy="0 0 0" />
-    </xacro:solid_cylinder_inertial>
-    <collision>
-      <origin xyz="0 0 0" rpy="0 0 0"/>
-      <geometry>
-        <cylinder length="${lidar_height}" radius="${lidar_radius}"/>
-      </geometry>
-    </collision>
-    <visual>
-      <origin xyz="0 0 0" rpy="0 0 0"/>
-      <geometry>
-        <cylinder length="${lidar_height}" radius="${lidar_radius}"/>
-      </geometry>
-    </visual>
-  </link>
-  <gazebo reference="lidar_link">
-    <material>Gazebo/Red</material>
-    <sensor type="ray" name="head_hokuyo_sensor">
-      <pose>0 0 0 0 0 0</pose>
-      <visualize>false</visualize>
-      <update_rate>40</update_rate>
-      <ray>
-        <scan>
-          <horizontal>
-            <samples>720</samples>
-            <resolution>1</resolution>
-            <min_angle>-3.14</min_angle>
-            <max_angle>3.14</max_angle>
-          </horizontal>
-        </scan>
-        <range>
-          <min>0.10</min>
-          <max>30.0</max>
-          <resolution>0.01</resolution>
-        </range>
-        <noise>
-          <type>gaussian</type>
-          <mean>0.0</mean>
-          <stddev>0.01</stddev>
-        </noise>
-      </ray>
-      <plugin name="gazebo_ros_head_hokuyo_controller" filename="libgazebo_ros_laser.so">
-        <topicName>/eSAUl/laser/scan</topicName>
-        <frameName>laser_frame</frameName>
-      </plugin>
-    </sensor>
-  </gazebo>
-  <joint name="lidar_joint" type="fixed">
-    <axis xyz="0 1 0" />
-    <origin xyz="0 0 ${chassis_height/2 + lidar_height/2}" rpy="0 0 0"/>
-    <parent link="base_link"/>
-    <child link="lidar_link"/>
-  </joint>
- <xacro:macro name="support_wheel" params="parent location *origin">
-    <link name="support_wheel_${location}_link">
-      <visual>
-        <origin xyz="0 0 0" rpy="0 0 0" />
-        <geometry>
-          <mesh filename="package://caster_description/mesh/support_wheel.stl" />
-        </geometry>
-        <material name="">
-          <color rgba="0.3 0.3 0.3 1.0" />>
-        </material>
-      </visual>
-      <collision>
-        <origin xyz="0 0 0" rpy="0 0 0" />
-        <geometry>
-          <mesh filename="package://caster_description/mesh/support_wheel.stl" />
-        </geometry>
-      </collision>
-      <xacro:default_inertial mass="5" />
-    </link>
-    <joint name="support_wheel_${location}_joint" type="fixed">
-      <xacro:insert_block name="origin" />
-      <parent link="${parent}" />
-      <child link="support_wheel_${location}_link" />
-      <!-- <axis xyz="0 0 1" /> -->
-    </joint>
-  </xacro:macro>
   <xacro:link_track name="link_right" />
 	<xacro:joint_track name="joint_right" child="link_right" origin_xyz="0 ${-chassis_width/2-box_width/1.5} ${-2*box_width}" />
@@ -262,5 +80,5 @@
   </xacro:support_wheel>
   <gazebo>
-    		<plugin name="ModelPlugin" filename="libesaul_description.so" >
+    		<plugin name="ModelPlugin" filename="libesaul_plugin.so" >
       		<robotName>eSAUl</robotName>
             <joint_left>joint_left_wheel</joint_left>

Commit message: ekf

File: esaul_description/urdf/esaul.xacro (robot description, xacro)
@@ -4,6 +4,7 @@
   <xacro:include filename="$(find esaul_description)/urdf/wheel.xacro" />
   <xacro:include filename="$(find esaul_description)/urdf/lidar.xacro" />
+  <xacro:include filename="$(find esaul_description)/urdf/imu.xacro" />
   <xacro:property name="M_PI" value="3.1415926535897931" />
-  <xacro:property name="chassis_mass" value="40" />
+  <xacro:property name="chassis_mass" value="20" />
   <xacro:property name="chassis_length" value="0.45" />
   <xacro:property name="chassis_width" value="0.22" />
@@ -68,14 +69,14 @@
 	<xacro:joint_wheel_left name="joint_left_wheel" child="left_wheel" origin_xyz="0 0 0" />
   <xacro:support_wheel parent="link_left" location="left_1">
-    <origin xyz="${box_length/2} 0 0.028" rpy="0 0 0" />
+    <origin xyz="${box_length/2} 0 0.02796" rpy="0 0 0" />
   </xacro:support_wheel>
   <xacro:support_wheel parent="link_left" location="left_2">
-    <origin xyz="${-box_length/2} 0 0.028" rpy="0 0 0" />
+    <origin xyz="${-box_length/2} 0 0.02796" rpy="0 0 0" />
   </xacro:support_wheel>
   <xacro:support_wheel parent="link_right" location="right_1">
-    <origin xyz="${box_length/2} 0 0.028" rpy="0 0 0" />
+    <origin xyz="${box_length/2} 0 0.02796" rpy="0 0 0" />
   </xacro:support_wheel>
   <xacro:support_wheel parent="link_right" location="right_2">
-    <origin xyz="${-box_length/2} 0 0.028" rpy="0 0 0" />
+    <origin xyz="${-box_length/2} 0 0.02796" rpy="0 0 0" />
   </xacro:support_wheel>
   <gazebo>

File: esaul_description/urdf/imu.xacro (robot description, xacro)
@@ -1,15 +1,54 @@
 <?xml version="1.0"?>
 <robot xmlns:xacro="http://www.ros.org/wiki/xacro">
+  <xacro:property name="imu_mass" value="0.01" />
+  <xacro:property name="imu_height" value="0.0002"/>
+  <xacro:property name="imu_radius" value="0.0004"/>
+  <xacro:property name="chassis_height" value="0.13" />
+  <xacro:macro name="solid_cylinder_inertial"
+               params="r h mass *origin">
+    <inertial>
+      <xacro:insert_block name="origin"/>
+      <mass value="${mass}"/>
+      <inertia ixx="${(mass * h * h)/12 + (mass * r * r)/4}" ixy="0.0" ixz="0.0"
+               iyy="${(mass * h * h)/12 + (mass * r * r)/4}" iyz="0.0"
+               izz="${mass / 2 * r * r}" />
+    </inertial>
+  </xacro:macro>
+ <link name="imu_link">
+    <xacro:solid_cylinder_inertial
+        r="${imu_radius}" h="${imu_height}"
+        mass="${imu_mass}" >
+      <origin xyz="0 0 0" rpy="0 0 0" />
+    </xacro:solid_cylinder_inertial>
+    <collision>
+      <origin xyz="0 0 0" rpy="0 0 0"/>
+      <geometry>
+        <cylinder length="${imu_height}" radius="${imu_radius}"/>
+      </geometry>
+    </collision>
+    <visual>
+      <origin xyz="0 0 0" rpy="0 0 0"/>
+      <geometry>
+        <cylinder length="${imu_height}" radius="${imu_radius}"/>
+      </geometry>
+    </visual>
+  </link>
   <gazebo>
-    <plugin filename="libcow_imu.so" name="imu_plugin">
-      <topicName>sensors/imu</topicName>
-      <serviceName>sensors/imu</serviceName>
-      <bodyName>base_link</bodyName>
-      <updateRateHZ>200.0</updateRateHZ>
-      <gaussianNoise>0.0</gaussianNoise>
-      <xyzOffset>0 0 0</xyzOffset>
-      <rpyOffset>0 0 0</rpyOffset>
-      <frameName>imu_link</frameName>
-    </plugin>
+      <plugin filename="libcow_imu.so" name="imu_plugin">
+        <topicName>eSAUl/imu</topicName>
+        <serviceName>eSAUl/service</serviceName>
+        <bodyName>base_link</bodyName>
+        <updateRateHZ>100.0</updateRateHZ>
+        <gaussianNoise>0</gaussianNoise>
+        <xyzOffset>0 0 0</xyzOffset>
+        <rpyOffset>0 0 0</rpyOffset>
+        <frameName>imu_link</frameName>
+      </plugin>
   </gazebo>
+  <joint name="imu_joint" type="fixed">
+    <axis xyz="0 1 0" />
+    <origin xyz="0 0 ${chassis_height/2}" rpy="0 0 0"/>
+    <parent link="base_link"/>
+    <child link="imu_link"/>
+  </joint>
 </robot>

File: esaul_description/urdf/lidar.xacro (robot description, xacro)
@@ -51,5 +51,5 @@
         <range>
           <min>0.10</min>
-          <max>30.0</max>
+          <max>10</max>
           <resolution>0.01</resolution>
         </range>
@@ -62,5 +62,5 @@
       <plugin name="gazebo_ros_head_hokuyo_controller" filename="libgazebo_ros_laser.so">
         <topicName>/eSAUl/laser/scan</topicName>
-        <frameName>laser_frame</frameName>
+        <frameName>lidar_link</frameName>
       </plugin>
     </sensor>

File: esaul_description/urdf/wheel.xacro (robot description, xacro)
@@ -1,5 +1,5 @@
 <?xml version="1.0"?>
 <robot xmlns:xacro="http://www.ros.org/wiki/xacro">
-  <xacro:property name="wheel_mass" value="10" />
+  <xacro:property name="wheel_mass" value="5" />
   <xacro:property name="track_rad" value="0.04" />
   <xacro:property name="track_length" value="0.03" />

Commit message: Kalman

File: esaul_description/urdf/esaul.xacro (robot description, xacro)
@@ -61,22 +61,22 @@
   </link>
   <xacro:link_track name="link_right" />
-	<xacro:joint_track name="joint_right" child="link_right" origin_xyz="0 ${-chassis_width/2-box_width/1.5} ${-2*box_width}" />
+	<xacro:joint_track name="joint_right" child="link_right" origin_xyz="0 ${-chassis_width/2-box_width/1.5} ${-2.1*box_width}" />
   <xacro:link_wheel name="right_wheel" />
 	<xacro:joint_wheel_right name="joint_right_wheel" child="right_wheel" origin_xyz="0 0 0" />
   <xacro:link_track name="link_left" />
-	<xacro:joint_track name="joint_left" child="link_left" origin_xyz="0 ${chassis_width/2+box_width/1.5} ${-2*box_width}" />
+	<xacro:joint_track name="joint_left" child="link_left" origin_xyz="0 ${chassis_width/2+box_width/1.5} ${-2.1*box_width}" />
   <xacro:link_wheel name="left_wheel" />
 	<xacro:joint_wheel_left name="joint_left_wheel" child="left_wheel" origin_xyz="0 0 0" />
   <xacro:support_wheel parent="link_left" location="left_1">
-    <origin xyz="${box_length/2} 0 0.02796" rpy="0 0 0" />
+    <origin xyz="${box_length/2} 0 0.027965" rpy="0 0 0" />
   </xacro:support_wheel>
   <xacro:support_wheel parent="link_left" location="left_2">
-    <origin xyz="${-box_length/2} 0 0.02796" rpy="0 0 0" />
+    <origin xyz="${-box_length/2} 0 0.027965" rpy="0 0 0" />
   </xacro:support_wheel>
   <xacro:support_wheel parent="link_right" location="right_1">
-    <origin xyz="${box_length/2} 0 0.02796" rpy="0 0 0" />
+    <origin xyz="${box_length/2} 0 0.027965" rpy="0 0 0" />
   </xacro:support_wheel>
   <xacro:support_wheel parent="link_right" location="right_2">
-    <origin xyz="${-box_length/2} 0 0.02796" rpy="0 0 0" />
+    <origin xyz="${-box_length/2} 0 0.027965" rpy="0 0 0" />
   </xacro:support_wheel>
   <gazebo>

File: esaul_description/urdf/imu.xacro (robot description, xacro)
@@ -1,54 +1,13 @@
 <?xml version="1.0"?>
 <robot xmlns:xacro="http://www.ros.org/wiki/xacro">
-  <xacro:property name="imu_mass" value="0.01" />
-  <xacro:property name="imu_height" value="0.0002"/>
-  <xacro:property name="imu_radius" value="0.0004"/>
-  <xacro:property name="chassis_height" value="0.13" />
-  <xacro:macro name="solid_cylinder_inertial"
-               params="r h mass *origin">
-    <inertial>
-      <xacro:insert_block name="origin"/>
-      <mass value="${mass}"/>
-      <inertia ixx="${(mass * h * h)/12 + (mass * r * r)/4}" ixy="0.0" ixz="0.0"
-               iyy="${(mass * h * h)/12 + (mass * r * r)/4}" iyz="0.0"
-               izz="${mass / 2 * r * r}" />
-    </inertial>
-  </xacro:macro>
- <link name="imu_link">
-    <xacro:solid_cylinder_inertial
-        r="${imu_radius}" h="${imu_height}"
-        mass="${imu_mass}" >
-      <origin xyz="0 0 0" rpy="0 0 0" />
-    </xacro:solid_cylinder_inertial>
-    <collision>
-      <origin xyz="0 0 0" rpy="0 0 0"/>
-      <geometry>
-        <cylinder length="${imu_height}" radius="${imu_radius}"/>
-      </geometry>
-    </collision>
-    <visual>
-      <origin xyz="0 0 0" rpy="0 0 0"/>
-      <geometry>
-        <cylinder length="${imu_height}" radius="${imu_radius}"/>
-      </geometry>
-    </visual>
-  </link>
   <gazebo>
-      <plugin filename="libcow_imu.so" name="imu_plugin">
-        <topicName>eSAUl/imu</topicName>
-        <serviceName>eSAUl/service</serviceName>
-        <bodyName>base_link</bodyName>
-        <updateRateHZ>100.0</updateRateHZ>
-        <gaussianNoise>0</gaussianNoise>
-        <xyzOffset>0 0 0</xyzOffset>
-        <rpyOffset>0 0 0</rpyOffset>
-        <frameName>imu_link</frameName>
-      </plugin>
+    <plugin name="imu_plugin" filename="libgazebo_ros_imu.so">
+      <alwaysOn>true</alwaysOn>
+      <bodyName>base_link</bodyName>
+      <topicName>/eSAUl/imu</topicName>
+      <serviceName>/eSAUl/service</serviceName>
+      <gaussianNoise>0.0</gaussianNoise>
+      <updateRate>50.0</updateRate>
+    </plugin>
   </gazebo>
-  <joint name="imu_joint" type="fixed">
-    <axis xyz="0 1 0" />
-    <origin xyz="0 0 ${chassis_height/2}" rpy="0 0 0"/>
-    <parent link="base_link"/>
-    <child link="imu_link"/>
-  </joint>
 </robot>
